File: newstuff/UHF_ANTENNA_6U_OFFICIAL/UHF_ANTENNA-6U/L1Band.kicad_sch (KiCad schematic)
At the start: 2 parts, among them J3 Conn_Coaxial, U1 GP.1575.15.4.B.02

Commit message: huifyt
vyuft
Parts:
- J3: footprint Connector_Coaxial:MMCX_Molex_73415-1471_Vertical -> Connector_Coaxial:WR-MMCX_Wuerth_66012102111404_Vertical
Changed lines of the file:
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@@
 			)
 		)
-		(property "Footprint" "Connector_Coaxial:MMCX_Molex_73415-1471_Vertical"
+		(property "Footprint" "Connector_Coaxial:WR-MMCX_Wuerth_66012102111404_Vertical"
 			(at 143.51 95.25 0)
 			(hide yes)
