File: newstuff/UHF_ANTENNA_6U_OFFICIAL/UHF_ANTENNA-6U/UHF.kicad_sch (KiCad schematic)
At the start: 11 parts, among them IC1 QBA-07+, IC2 QBA-07+, IC3 QBA-07+, J1 Conn_Coaxial

Commit message: huifyt
vyuft
Parts:
- removed AE2: Antenna, AntennaPads:TestPoint_Pad_4.0x4.0mm, symbol Device:Antenna
- added AE6: Antenna, AntennaPads:TestPoint_Pad_4.0x4.0mm, symbol Device:Antenna
- added H1, H2, H3, H4: MountingHole, MountingHole:MountingHole_3.2mm_M3, symbol Mechanical:MountingHole
- J1: footprint Connector_Coaxial:WR-MMCX_Wuerth_66012102111404_Vertical -> Connector_Coaxial:MMCX_Molex_73415-1471_Vertical
Connections:
- net at IC3.10 (PORT_1_(+90°)): now also AE6.1 (A); no longer AE4.1 (A)
- net at IC2.6 (PORT_2_(0°)): now also AE4.1 (A)
