File: newstuff/UHF_ANTENNA_6U_OFFICIAL/UHF_ANTENNA-6U/UHF_ANTENNA-6U.kicad_pcb (KiCad board)
At the start: 6 copper layers, 204 x 99.1 mm, 35 parts, among them IC1 QBA-07+, IC2 QBA-07+, IC3 QBA-07+, J1 Conn_Coaxial, J2 Conn_01x02, J27 USB_C_Receptacle_USB2.0_16P, J5 Conn_01x02, J6 Conn_01x02, Q1 IRLML2052, Q27 Q_PMOS_DGS, Q28 Q_PMOS_DGS, U11 CYPD3177-24LQ

Commit message: huifyt
vyuft
Parts:
- added H1: MountingHole, MountingHole:MountingHole_3.2mm_M3, F.Cu at (76.7, 37.3)
- added H2: MountingHole, MountingHole:MountingHole_3.2mm_M3, F.Cu at (76.7, 125.3)
- added H3: MountingHole, MountingHole:MountingHole_3.2mm_M3, F.Cu at (240.7, 37.3)
- added H4: MountingHole, MountingHole:MountingHole_3.2mm_M3, F.Cu at (240.7, 125.3)
- J1: footprint Connector_Coaxial:WR-MMCX_Wuerth_66012102111404_Vertical -> Connector_Coaxial:MMCX_Molex_73415-1471_Vertical
- J27: moved to B.Cu
- turned J27 to 0 degrees
Connections:
- IC2 pad 6: Net-(AE2-A) -> Net-(AE4-A)
- IC3 pad 10: Net-(AE4-A) -> Net-(AE6-A)
Routing:
- net Net-(AE5-A): track 48.9 -> 52.4 mm
- net Net-(AE4-A): track 49.0 -> 52.5 mm
- net CC1: track 31.5 -> 28.2 mm, vias 2 -> 1
- net CC2: track 35.5 -> 38.4 mm, vias 2 -> 1
- net Net-(AE3-A): track 43.2 -> 41.3 mm
Other:
- board text added: "9/10/2025"
- board text added: "ANTENNA BOARD REV1 KAUSHIQE DAMEAN QAREEM BRIGHTON RIVERA #1 (ANTONIO) RIVERA #2 (LUIGI) OCTABLO KACHOW PIPLUP PLUSHDEGREE"
- board text added: "H1"
- board text removed: "ANTENNA BOARD REV1 KAUSHIQE DAMEAN MUDTIN"
