File: oldstuff/UHF_ANTENNA_6U_OFFICIAL/UHF_ANTENNA-6U/UHF_ANTENNA-6U.kicad_pcb (KiCad board)
At the start: 4 copper layers, 204 x 99.1 mm, 38 parts, among them IC1 QBA-07+, IC2 QBA-07+, IC3 QBA-07+, J1 Conn_Coaxial, J2 Conn_01x02, J27 USB_C_Receptacle_USB2.0_16P, J3 Conn_Coaxial, J5 Conn_01x02, J6 Conn_01x02, Q1 IRLML0030, Q27 Q_PMOS_DGS, Q28 Q_PMOS_DGS, U1 GP.1575.15.4.B.02, U11 CYPD3177-24LQ

Commit message: huifyt
vyuft
Parts:
- moved R5 51.4 mm to (190.5, 93.8)
Routing:
- net VSS: vias 710 -> 711
Changed lines of the file:
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@@
 	(footprint "PAC:PAC01_VIS"
 		(layer "F.Cu")
-		(at 153.192604 58.432604 -45)
+		(at 190.462604 93.812604 -45)
 		(tags "PAC100003009FA1000 ")
 		(property "Reference" "R5"
@@
 	)
 	(via
+		(at 129.5 76.82)
+		(size 0.6)
+		(drill 0.3)
+		(layers "F.Cu" "B.Cu")
+		(free yes)
+		(net "VSS")
+	)
+	(via
 		(at 200.764039 66.283994)
 		(size 0.6)
@@
 		(net "VSS")
 	)
+	(via
+		(at 118.29 57.41875)
+		(size 0.6)
+		(drill 0.3)
+		(layers "F.Cu" "B.Cu")
+		(net "/BurnWire/12VINP")
+	)
+	(segment
+		(start 118.24 51.99125)
+		(end 118.24 57.36875)
+		(width 1)
+		(layer "In1.Cu")
+		(net "/BurnWire/12VINP")
+	)
+	(segment
+		(start 118.24 57.36875)
+		(end 118.29 57.41875)
+		(width 1)
+		(layer "In1.Cu")
+		(net "/BurnWire/12VINP")
+	)
+	(via
+		(at 232.97 106.425)
+		(size 0.6)
+		(drill 0.3)
+		(layers "F.Cu" "B.Cu")
+		(net "Net-(Q1-D)")
+	)
 	(segment
 		(start 89.33 49.89)
@@
 	)
 	(segment
+		(start 237.56 107.83)
+		(end 237.56 106.47)
+		(width 1)
+		(layer "F.Cu")
+		(net "Net-(Q1-G)")
+	)
+	(segment
+		(start 235.64 104.55)
+		(end 233.92 104.55)
+		(width 1)
+		(layer "F.Cu")
+		(net "Net-(Q1-G)")
+	)
+	(segment
+		(start 237.56 106.47)
+		(end 235.64 104.55)
+		(width 1)
+		(layer "F.Cu")
+		(net "Net-(Q1-G)")
+	)
+	(segment
 		(start 84.9965 42.9955)
 		(end 84.9965 46.5175)
@@
 		(net "Net-(U11-ISNK_COARSE)")
 	)
+	(segment
+		(start 239.28 107.9)
+		(end 239.21 107.83)
+		(width 1)
+		(layer "F.Cu")
+		(net "Net-(J6-Pin_2)")
+	)
+	(segment
+		(start 239.28 113.34)
+		(end 239.28 107.9)
+		(width 1)
+		(layer "F.Cu")
+		(net "Net-(J6-Pin_2)")
+	)
 	(via
 		(at 83.985 50.23)
@@
 	)
 	(segment
+		(start 174.16 81.29)
+		(end 158.5985 81.29)
+		(width 0.3203)
+		(layer "F.Cu")
+		(net "Net-(J3-In)")
+	)
+	(segment
+		(start 158.5985 81.29)
+		(end 158.5925 81.284)
+		(width 0.3203)
+		(layer "F.Cu")
+		(net "Net-(J3-In)")
+	)
+	(segment
 		(start 141.951807 86.626399)
 		(end 141.793809 86.784398)
@@
 		(net "Net-(AE5-A)")
 	)
-	(via
-		(at 118.29 57.41875)
-		(size 0.6)
-		(drill 0.3)
-		(layers "F.Cu" "B.Cu")
-		(net "/BurnWire/12VINP")
-	)
-	(segment
-		(start 118.24 51.99125)
-		(end 118.24 57.36875)
-		(width 1)
-		(layer "In1.Cu")
-		(net "/BurnWire/12VINP")
-	)
-	(segment
-		(start 118.24 57.36875)
-		(end 118.29 57.41875)
-		(width 1)
-		(layer "In1.Cu")
-		(net "/BurnWire/12VINP")
-	)
-	(segment
-		(start 239.28 107.9)
-		(end 239.21 107.83)
-		(width 1)
-		(layer "F.Cu")
-		(net "Net-(J6-Pin_2)")
-	)
-	(segment
-		(start 239.28 113.34)
-		(end 239.28 107.9)
-		(width 1)
-		(layer "F.Cu")
-		(net "Net-(J6-Pin_2)")
-	)
-	(segment
-		(start 237.56 107.83)
-		(end 237.56 106.47)
-		(width 1)
-		(layer "F.Cu")
-		(net "Net-(Q1-G)")
-	)
-	(segment
-		(start 235.64 104.55)
-		(end 233.92 104.55)
-		(width 1)
-		(layer "F.Cu")
-		(net "Net-(Q1-G)")
-	)
-	(segment
-		(start 237.56 106.47)
-		(end 235.64 104.55)
-		(width 1)
-		(layer "F.Cu")
-		(net "Net-(Q1-G)")
-	)
-	(via
-		(at 232.97 106.425)
-		(size 0.6)
-		(drill 0.3)
-		(layers "F.Cu" "B.Cu")
-		(net "Net-(Q1-D)")
-	)
-	(segment
-		(start 174.16 81.29)
-		(end 158.5985 81.29)
-		(width 0.3203)
-		(layer "F.Cu")
-		(net "Net-(J3-In)")
-	)
-	(segment
-		(start 158.5985 81.29)
-		(end 158.5925 81.284)
-		(width 0.3203)
-		(layer "F.Cu")
-		(net "Net-(J3-In)")
-	)
 	(zone
