File: newstuff/UHF_ANTENNA_6U_OFFICIAL/UHF_ANTENNA-6U/UHF_ANTENNA-6U-2026-09-10_114102/.history/PowerTransfer.kicad_sch (KiCad schematic)
At the start: 19 parts, among them J2 Conn_01x02, J27 USB_C_Receptacle_USB2.0_16P, Q27 Q_PMOS_DGS, Q28 Q_PMOS_DGS, U11 CYPD3177-24LQ

Commit message: changes
changes
Parts:
- J27: footprint Connector_USB:USB_C_Receptacle_GCT_USB4110 -> Connector_USB:USB_C_Receptacle_HRO_TYPE-C-31-M-12
Changed lines of the file:
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@@
 			)
 		)
-		(property "Footprint" "Connector_USB:USB_C_Receptacle_GCT_USB4110"
+		(property "Footprint" "Connector_USB:USB_C_Receptacle_HRO_TYPE-C-31-M-12"
 			(at 107.95 111.76 0)
 			(hide yes)
