File: newstuff/UHF_ANTENNA_6U_OFFICIAL/UHF_ANTENNA-6U/UHF_ANTENNA-6U-2026-09-10_114102/.history/resistor.kicad_sch (KiCad schematic)
At the start: 6 parts, among them J5 Conn_01x02, J6 Conn_01x02, Q1 IRLML2052

Commit message: changes
changes
Parts:
- J5: footprint XH-2A:JST_B2B-XH-A -> TerminalBlock_RND:TerminalBlock_RND_205-00276_1x02_P5.00mm_Vertical
- J6: footprint Connector_PinSocket_2.54mm:PinSocket_1x02_P2.54mm_Vertical_SMD_Pin1Left -> TerminalBlock_RND:TerminalBlock_RND_205-00276_1x02_P5.00mm_Vertical
Connections:
- net 12VINP: now also R5.1; no longer R5.2
- net at Q1.3 (D): now also R5.2; no longer R5.1
Other:
- moved on the sheet: R5
Changed lines of the file:
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@@
 	(symbol
 		(lib_id "plusz-end-card-with-turnstile-eagle-import:PAC100-FOR-MELTWIRE")
-		(at 153.67 90.17 90)
+		(at 153.67 90.17 270)
 		(unit 1)
 		(body_style 1)
@@
 		(dnp no)
 		(property "Reference" "R5"
-			(at 152.1714 93.98 0)
+			(at 155.1686 86.36 0)
 			(show_name no)
 			(do_not_autoplace no)
@@
 		)
 		(property "Value" "7.5  1W"
-			(at 156.972 95.25 0)
+			(at 150.368 85.09 0)
 			(show_name no)
 			(do_not_autoplace no)
@@
 		)
 		(property "Footprint" "PAC:PAC01_VIS"
-			(at 146.558 89.154 0)
+			(at 160.782 91.186 0)
 			(hide yes)
 			(show_name no)
@@
 			)
 		)
-		(property "Footprint" "XH-2A:JST_B2B-XH-A"
+		(property "Footprint" "TerminalBlock_RND:TerminalBlock_RND_205-00276_1x02_P5.00mm_Vertical"
 			(at 153.67 48.26 0)
 			(hide yes)
@@
 			)
 		)
-		(property "Footprint" "Connector_PinSocket_2.54mm:PinSocket_1x02_P2.54mm_Vertical_SMD_Pin1Left"
+		(property "Footprint" "TerminalBlock_RND:TerminalBlock_RND_205-00276_1x02_P5.00mm_Vertical"
 			(at 110.49 125.73 0)
 			(hide yes)
