File: newstuff/UHF_ANTENNA_6U_OFFICIAL/UHF_ANTENNA-6U/UHF_ANTENNA-6U-2026-09-10_114102/UHF_ANTENNA-6U-backups/UHF_ANTENNA-6U-2026-09-05_155604/PowerTransfer.kicad_sch (KiCad schematic)
At the start: 19 parts, among them J2 Conn_01x02, J27 USB_C_Receptacle_USB2.0_16P, Q27 Q_PMOS_DGS, Q28 Q_PMOS_DGS, U11 CYPD3177-24LQ

Commit message: changes
changes
Parts:
- removed J2: Conn_01x02, TerminalBlock_RND:TerminalBlock_RND_205-00276_1x02_P5.00mm_Vertical, symbol Connector_Generic:Conn_01x02
- J27: footprint Connector_USB:USB_C_Receptacle_GCT_USB4110 -> Connector_USB:USB_C_Receptacle_HRO_TYPE-C-31-M-12
Connections:
- net VBUS: now also Q27.1 (D); no longer Q27.3 (D)
- net VDC_OUT: now also Q28.1 (D); no longer Q28.3 (D)
- net VDDD: no longer R75.1
- net at C56.2, C58.2, R69.2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: now also Q27.2 (G), Q28.2 (G); no longer Q27.1 (G), Q28.1 (G)
- new net: Q27.3 (S), Q28.3 (S), R73.1
- new net +3.3V: R75.1
