File: newstuff/UHF_ANTENNA-6U-OFFICIAL/UHF_ANTENNA-6U.kicad_pcb (KiCad board)
At the start: 6 copper layers, 206 x 99.1 mm, 43 parts, among them IC1 QBA-07+, IC2 QBA-07+, IC3 QBA-07+, J1 Conn_Coaxial, J2 Conn_01x02, J27 USB_C_Receptacle_USB2.0_16P, J3 Conn_Coaxial, J5 Conn_01x02, J6 Conn_01x02, Q1 IRLML2052, Q27 Q_PMOS_DGS, Q28 Q_PMOS_DGS, U11 CYPD3177-24LQ

Commit message: changes
cleaning up stuff
Routing:
- net VDDD: track 15.9 -> 29.4 mm
- net VBUS: track 18.6 -> 23.5 mm, vias 1 -> 3
- net VSS: track 4.99 -> 7.06 mm, vias 816 -> 817
- net Net-(IC1-SUM_PORT): track 8.10 -> 8.06 mm, vias 1 -> 0
Changed lines of the file:
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@@
 	)
 	(segment
-		(start 120.95 63.7)
-		(end 127.379 57.271)
+		(start 138.734 78.25)
+		(end 122.5 78.25)
 		(width 1)
 		(layer "In3.Cu")
@@
 	)
 	(segment
-		(start 130.877 54.377)
-		(end 130.9 54.4)
+		(start 120.95 76.7)
+		(end 120.95 63.7)
 		(width 1)
 		(layer "In3.Cu")
@@
 	)
 	(segment
-		(start 120.95 76.7)
-		(end 120.95 63.7)
+		(start 130.877 54.377)
+		(end 130.9 54.4)
 		(width 1)
 		(layer "In3.Cu")
@@
 	)
 	(segment
-		(start 122.75 78.5)
+		(start 122.5 78.25)
 		(end 120.95 76.7)
 		(width 1)
@@
 	)
 	(segment
-		(start 138.484 78.5)
-		(end 122.75 78.5)
+		(start 120.95 63.7)
+		(end 127.379 57.271)
 		(width 1)
 		(layer "In3.Cu")
@@
 	(segment
 		(start 141.470793 75.513207)
-		(end 138.484 78.5)
+		(end 138.734 78.25)
 		(width 1)
 		(layer "In3.Cu")
@@
 	)
 	(via
+		(at 124.5 79.5)
+		(size 0.6)
+		(drill 0.3)
+		(layers "F.Cu" "B.Cu")
+		(free yes)
+		(net "VSS")
+	)
+	(via
 		(at 142.684842 67.1057)
 		(size 0.6)
@@
 	)
 	(via
-		(at 126 80.75)
+		(at 126.005 80.848)
 		(size 0.6)
 		(drill 0.3)
@@
 	)
 	(via
+		(at 125.5 79.5)
+		(size 0.6)
+		(drill 0.3)
+		(layers "F.Cu" "B.Cu")
+		(free yes)
+		(net "VSS")
+	)
+	(via
 		(at 123.75 77)
 		(size 0.6)
@@
 	)
 	(via
-		(at 126 79.75)
+		(at 126.25 80)
 		(size 0.6)
 		(drill 0.3)
@@
 	)
 	(via
-		(at 104.5 53.18)
-		(size 0.6)
-		(drill 0.3)
-		(layers "F.Cu" "B.Cu")
-		(free yes)
-		(net "VSS")
-	)
-	(via
 		(at 202.180683 67.880138)
 		(size 0.6)
@@
 	)
 	(via
-		(at 123.5 79.75)
+		(at 123.5 79.5)
 		(size 0.6)
 		(drill 0.3)
@@
 		(net "VSS")
 	)
+	(segment
+		(start 91.159 52.431)
+		(end 90.909 52.681)
+		(width 0.3)
+		(layer "B.Cu")
+		(net "VSS")
+	)
+	(segment
+		(start 90.909 52.681)
+		(end 90.909 54.406)
+		(width 0.3)
+		(layer "B.Cu")
+		(net "VSS")
+	)
 	(via
 		(at 237.664 105.873)
@@
 	)
 	(segment
-		(start 211.41 99.89)
-		(end 211.44 99.92)
-		(width 0.2214)
-		(layer "F.Cu")
-		(net "Net-(IC1-SUM_PORT)")
-	)
-	(via
-		(at 211.44 99.92)
-		(size 0.6)
-		(drill 0.3)
-		(layers "F.Cu" "B.Cu")
-		(net "Net-(IC1-SUM_PORT)")
-	)
-	(segment
 		(start 206.44 94.81)
 		(end 206.49 94.76)
@@
 	)
 	(segment
-		(start 90.521 55.499)
-		(end 93.712 55.499)
-		(width 1)
-		(layer "F.Cu")
-		(net "VDDD")
-	)
-	(segment
 		(start 93.712 55.499)
 		(end 93.729 55.516)
@@
 	)
 	(segment
+		(start 93.729 57.036)
+		(end 93.729 55.516)
+		(width 1)
+		(layer "In3.Cu")
+		(net "VDDD")
+	)
+	(segment
 		(start 85.277 53.644)
 		(end 85.939 54.306)
@@
 	)
 	(segment
+		(start 93.712 55.499)
+		(end 93.729 55.516)
+		(width 1)
+		(layer "In3.Cu")
+		(net "VDDD")
+	)
+	(segment
+		(start 92.129 58.636)
+		(end 93.729 57.036)
+		(width 1)
+		(layer "In3.Cu")
+		(net "VDDD")
+	)
+	(segment
+		(start 85.939 57.151)
+		(end 87.424 58.636)
+		(width 1)
+		(layer "In3.Cu")
+		(net "VDDD")
+	)
+	(segment
 		(start 85.277 48.143)
 		(end 85.277 53.644)
@@
 		(net "VDDD")
 	)
+	(segment
+		(start 85.939 54.306)
+		(end 85.939 57.151)
+		(width 1)
+		(layer "In3.Cu")
+		(net "VDDD")
+	)
+	(segment
+		(start 90.521 55.499)
+		(end 93.712 55.499)
+		(width 1)
+		(layer "In3.Cu")
+		(net "VDDD")
+	)
+	(segment
+		(start 87.424 58.636)
+		(end 92.129 58.636)
+		(width 1)
+		(layer "In3.Cu")
+		(net "VDDD")
+	)
 	(via
 		(at 94.988 47.007)
@@
 	)
 	(via
-		(at 95.294 52.591)
-		(size 0.6)
+		(at 97.219 40.776)
+		(size 0.5)
+		(drill 0.3)
+		(layers "F.Cu" "B.Cu")
+		(net "VBUS")
+	)
+	(via
+		(at 97.523 38.522)
+		(size 0.5)
+		(drill 0.3)
+		(layers "F.Cu" "B.Cu")
+		(net "VBUS")
+	)
+	(via
+		(at 92.623 38.522)
+		(size 0.5)
 		(drill 0.3)
 		(layers "F.Cu" "B.Cu")
@@
 	)
 	(segment
-		(start 97.523 40.472)
-		(end 97.219 40.776)
-		(width 0.6)
+		(start 94.011944 53.681)
+		(end 95.197972 52.494972)
+		(width 0.3)
 		(layer "B.Cu")
 		(net "VBUS")
@@
 	(segment
 		(start 93.134 53.681)
-		(end 93.619096 53.681)
+		(end 94.011944 53.681)
 		(width 0.3)
 		(layer "B.Cu")
@@
 	)
 	(segment
-		(start 94.709096 52.591)
-		(end 95.294 52.591)
-		(width 0.3)
-		(layer "B.Cu")
-		(net "VBUS")
-	)
-	(segment
 		(start 95.676944 52.016)
 		(end 95.197972 52.494972)
@@
 	)
 	(segment
-		(start 97.523 38.522)
-		(end 97.523 40.472)
-		(width 0.6)
-		(layer "B.Cu")
-		(net "VBUS")
-	)
-	(segment
 		(start 96.365284 51.950716)
 		(end 95.812938 51.950716)
@@
 	)
 	(segment
-		(start 93.619096 53.681)
-		(end 94.709096 52.591)
-		(width 0.3)
-		(layer "B.Cu")
-		(net "VBUS")
-	)
-	(segment
 		(start 97.119 47.336)
 		(end 97.119 51.197)
@@
 		(net "VBUS")
 	)
+	(segment
+		(start 97.523 38.522)
+		(end 97.523 40.472)
+		(width 1)
+		(layer "In3.Cu")
+		(net "VBUS")
+	)
+	(segment
+		(start 97.523 40.472)
+		(end 97.219 40.776)
+		(width 1)
+		(layer "In3.Cu")
+		(net "VBUS")
+	)
+	(segment
+		(start 92.623 38.522)
+		(end 97.523 38.522)
+		(width 1)
+		(layer "In3.Cu")
+		(net "VBUS")
+	)
 	(via
 		(at 100.997 49.038)
@@
 	(segment
 		(start 95.145 50.351)
-		(end 96.76 48.736)
+		(end 95.94 49.556)
 		(width 0.3)
 		(layer "In2.Cu")
@@
 	)
 	(segment
-		(start 96.76 48.736)
+		(start 95.94 49.556)
+		(end 95.94 37.34)
+		(width 0.3)
+		(layer "In2.Cu")
+		(net "CC2")
+	)
+	(segment
+		(start 95.94 37.34)
 		(end 96.76 36.52)
 		(width 0.3)
